File: PCB/Cabinas/Cabinas.sch (KiCad schematic (older format))
At the start: 115 parts, among them J1 JACK_ST_3SW, K1 CONN_3, M1 WTV020-SD, P1 CONN_2, P10 CONN_2, P11 CONN_2, P12 CONN_2, P13 DIN_5, P2 CONN_2, P3 CONN_2, P4 CONN_2, P5 CONN_2, P6 CONN_2, P7 CONN_2, P8 CONN_2, P9 CONN_2, Q1 MOSFET_N, Q10 MOSFET_N, Q11 MOSFET_N, Q12 MOSFET_N, Q2 MOSFET_N, Q3 MOSFET_N, Q4 MOSFET_N, Q5 MOSFET_N, Q6 MOSFET_N, Q7 MOSFET_N, Q8 MOSFET_N, Q9 MOSFET_N, SW1 PUSHBUTTON, SW10 PUSHBUTTON, SW11 PUSHBUTTON, SW12 PUSHBUTTON, SW2 PUSHBUTTON, SW3 PUSHBUTTON, SW4 PUSHBUTTON, SW5 PUSHBUTTON, SW6 PUSHBUTTON, SW7 PUSHBUTTON, SW8 PUSHBUTTON, SW9 PUSHBUTTON, U1 BTM, U2 7805, U3 TL072, U4 74HC595, U5 74HC595

Commit message: Revision final
Revision final
Parts:
- removed C13: 470uF, ~, symbol CP1
- removed GS1, GS2: GS3, symbol GS3
- removed U4, U5: 74HC595, ~, symbol 74HC595
Connections:
- net labels added: D10, D11, D12, D13, D2, D3, D5, D6, D7, D8, D9
- net labels removed: 1, 10, 11, 12, 2, 3, 4, 5, 6, 7, 8, 9, SR_CLK, SR_Input, SR_LCLK, SR_OE
- wire segments 429 -> 375
- no-connect marks 19 -> 12
Other:
- note removed: "Shift register"
- moved on the sheet: A1, C1, C10, C11, C12, C2, C3, C4, C5, C6, C7, C8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

Commit message: Cambios
Cambio en los capacitores de desacoplamiento y sus footprints.
Parts:
- added C13: 470uF, ~, symbol CP1
- added GS1: GS3, symbol GS3
Connections:
- wire segments 375 -> 381
Other:
- moved on the sheet: C3, C4, C5, C6, C7, C8, R18, R19

Commit message: Cambios
Cambio de pines para el módulo MP3
Parts:
- added GS2: GS3, symbol GS3
Connections:
- wire segments 381 -> 377
- no-connect marks 12 -> 15

Commit message: Shift registers
Se añadieron shift registers
Parts:
- added U4, U5: 74HC595, ~, symbol 74HC595
Connections:
- net labels added: 1, 10, 11, 12, 2, 3, 4, 5, 6, 7, 8, 9, SR_CLK, SR_Input, SR_LCLK, SR_OE
- net labels removed: D10, D11, D12, D13, D2, D3, D5, D6, D7, D8, D9
- wire segments 377 -> 429
- no-connect marks 15 -> 19
Other:
- note added: "Shift register"
- moved on the sheet: A1, C1, C10, C11, C12, C13, C2, C3, C4, C5, C6, C7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
